Commit message: Gripper width taken from detection

File: workspace/src/smart_robotics/urdf/red_cylinder.urdf (robot description, URDF)
Before this commit: robot red_cube, 1 links, 0 joints
Links:
- link base_link: geometry collision cylinder length=0.1 radius=0.03; visual cylinder length=0.1 radius=0.03

File: workspace/src/smart_robotics/urdf/red_rectangle.urdf (robot description, URDF)
Before this commit: robot red_cube, 1 links, 0 joints
Links:
- link base_link: geometry collision box size=0.12 0.06 0.06; visual box size=0.12 0.06 0.06
